File: k8split-PCB/k8split.kicad_pcb (KiCad board)
At the start: 2 copper layers, 397.3 x 124 mm, 245 parts, among them J1 AVR-ISP-6, J2 AVR-ISP-6, J3 Breakaway_Tabs, J4 Breakaway_Tabs, J5 Breakaway_Tabs, J6 Breakaway_Tabs, J7 Breakaway_Tabs, J8 Breakaway_Tabs, J9 Breakaway_Tabs, SW1 SW_Push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

Commit message: more trace cleanup
Parts:
- moved C3 1.74 mm to (20.1, 134.1), turned to 180 degrees
- moved C6 1.08 mm to (37.3, 128.8), turned to 90 degrees
- moved C7 0.92 mm to (25.9, 124.2), turned to 90 degrees
- moved C5 0.25 mm to (204.5, 128.0)
Routing:
- net COL7-R: track 230.0 -> 234.5 mm
- net COL6-R: track 219.9 -> 222.5 mm
- net COL2: track 159.3 -> 161.8 mm
- net COL1: track 178.3 -> 180.8 mm
- net COL0: track 194.4 -> 196.7 mm
- net +5VA: track 342.6 -> 340.3 mm
- net +5V: track 334.5 -> 336.3 mm
- net Net-(C3-Pad1): track 5.12 -> 3.82 mm
- net RESET: track 120.0 -> 120.7 mm
- net GND: vias 5 -> 4
