File: k8split-PCB/k8split.kicad_sch (KiCad schematic)
At the start: 227 parts, among them J1 DE15_Socket_HighDensity_Mount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, J10 Breakaway_Tabs, J11 DE15_Socket_HighDensity_Mount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, J12 DE15_Socket_HighDensity_Mount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, J2 DE15_Socket_HighDensity_Mount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, J3 Breakaway_Tabs, J4 Breakaway_Tabs, J5 Breakaway_Tabs, J6 Breakaway_Tabs, J7 Breakaway_Tabs, J8 Breakaway_Tabs, J9 Breakaway_Tabs, SW1 SW_Push, U1 ATmega32U4-AU, Y1 16MHz

Commit message: final order data update
Parts:
- removed J5, J6: Breakaway_Tabs, locallib:breakaway-mousebites, symbol Connector_Generic:Conn_01x01
Connections:
- no-connect marks 12 -> 10
Changed lines of the file:
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@@
 	)
 	(no_connect
-		(at 147.32 153.67)
-	)
-	(no_connect
 		(at 146.685 173.355)
 	)
 	(no_connect
-		(at 147.32 149.225)
-	)
-	(no_connect
 		(at 104.14 95.25)
 	)
@@
 					(unit 1)
 				)
-			)
-		)
-	)
-	(symbol
-		(lib_id "Connector_Generic:Conn_01x01")
-		(at 152.4 153.67 0)
-		(unit 1)
-		(body_style 1)
-		(exclude_from_sim no)
-		(in_bom yes)
-		(on_board yes)
-		(in_pos_files yes)
-		(dnp no)
-		(property "Reference" "J6"
-			(at 154.4066 152.6032 0)
-			(show_name no)
-			(do_not_autoplace no)
-			(effects
-				(font
-					(size 1.27 1.27)
-				)
-				(justify left)
-			)
-		)
-		(property "Value" "Breakaway_Tabs"
-			(at 154.4066 154.9146 0)
-			(show_name no)
-			(do_not_autoplace no)
-			(effects
-				(font
-					(size 1.27 1.27)
-				)
-				(justify left)
-			)
-		)
-		(property "Footprint" "locallib:breakaway-mousebites"
-			(at 152.4 153.67 0)
-			(hide yes)
-			(show_name no)
-			(do_not_autoplace no)
-			(effects
-				(font
-					(size 1.27 1.27)
-				)
-			)
-		)
-		(property "Datasheet" "~"
-			(at 152.4 153.67 0)
-			(hide yes)
-			(show_name no)
-			(do_not_autoplace no)
-			(effects
-				(font
-					(size 1.27 1.27)
-				)
-			)
-		)
-		(property "Description" ""
-			(at 152.4 153.67 0)
-			(show_name no)
-			(do_not_autoplace no)
-			(effects
-				(font
-					(size 1.27 1.27)
-				)
-			)
-		)
-		(pin "1"
-		)
-		(instances
-			(project "k8split"
-				(path "/d44da92a-04f6-4bc9-b452-5e8f1c673a7c"
-					(reference "J6")
-					(unit 1)
-				)
-			)
-		)
-	)
-	(symbol
-		(lib_id "Connector_Generic:Conn_01x01")
-		(at 152.4 149.225 0)
-		(unit 1)
-		(body_style 1)
-		(exclude_from_sim no)
-		(in_bom yes)
-		(on_board yes)
-		(in_pos_files yes)
-		(dnp no)
-		(property "Reference" "J5"
-			(at 154.4066 148.1582 0)
-			(show_name no)
-			(do_not_autoplace no)
-			(effects
-				(font
-					(size 1.27 1.27)
-				)
-				(justify left)
-			)
-		)
-		(property "Value" "Breakaway_Tabs"
-			(at 154.4066 150.4696 0)
-			(show_name no)
-			(do_not_autoplace no)
-			(effects
-				(font
-					(size 1.27 1.27)
-				)
-				(justify left)
-			)
-		)
-		(property "Footprint" "locallib:breakaway-mousebites"
-			(at 152.4 149.225 0)
-			(hide yes)
-			(show_name no)
-			(do_not_autoplace no)
-			(effects
-				(font
-					(size 1.27 1.27)
-				)
-			)
-		)
-		(property "Datasheet" "~"
-			(at 152.4 149.225 0)
-			(hide yes)
-			(show_name no)
-			(do_not_autoplace no)
-			(effects
-				(font
-					(size 1.27 1.27)
-				)
-			)
-		)
-		(property "Description" ""
-			(at 152.4 149.225 0)
-			(show_name no)
-			(do_not_autoplace no)
-			(effects
-				(font
-					(size 1.27 1.27)
-				)
-			)
-		)
-		(pin "1"
-		)
-		(instances
-			(project "k8split"
-				(path "/d44da92a-04f6-4bc9-b452-5e8f1c673a7c"
-					(reference "J5")
-					(unit 1)
-				)
